Commit message: 6-18 wipe blackboard runnable

File: fmauch_universal_robot/ur_e_description/urdf/ur5e.urdf.xacro (robot description, xacro)
@@ -308,5 +308,7 @@
       <parent link="${prefix}wrist_3_link" />
       <child link = "${prefix}ee_link" />
-      <origin xyz="0.0 0.0 0.0" rpy="0.0 ${-pi/2.0} ${pi/2.0}" />
+      <origin xyz="0.0 0.0 0.12" rpy="${-pi} 0.0 ${-pi/2.0}" />
+      <!-- <origin xyz="0.0 0.0 0.165" rpy="${-pi} 0.0 ${-pi/2.0}" /> -->
+      <!-- <origin xyz="0.0 0.0 0.165" rpy="0.0 ${-pi/2.0} ${pi/2.0}" /> -->
     </joint>
     <link name="${prefix}ee_link">
